Commit message: updated code

File: obot_description/urdf/color_macros.xacro (robot description, xacro)
@@ -1,24 +1,38 @@
 <?xml version="1.0"?>
 <robot xmlns:xacro="http://www.ros.org/wiki/xacro" >
-    <material name="white">
-        <color rgba="1 1 1 1" />
-    </material>
-    <material name="grey">
-        <color rgba="0.25 0.25 0.25 1"/>
-    </material>
-    <material name="orange">
-        <color rgba="1 0.55 0 1"/>
-    </material>
-    <material name="blue">
-        <color rgba="0.2 0.2 1 1"/>
-    </material>
-    <material name="red">
-        <color rgba="1 0 0 1"/>
-    </material>
-    <material name="black">
-        <color rgba="0.1 0.1 0.1 1"/>
-    </material>
-    <material name="silver">
-        <color rgba="0.6 0.6 0.6 1"/>
-    </material>
+    <xacro:macro name="material_blue">
+        <material name="blue">
+            <color rgba="0.2 0.2 1 1"/>
+        </material>
+    </xacro:macro>
+    <xacro:macro name="material_white">
+        <material name="white">
+            <color rgba="0.955 0.955 0.955 1"/>
+        </material>
+    </xacro:macro>
+    <xacro:macro name="material_grey">
+        <material name="grey">
+            <color rgba="0.3 0.3 0.3 1"/>
+        </material>
+    </xacro:macro>
+    <xacro:macro name="material_orange">
+        <material name="orange">
+            <color rgba="1 0.5 0 1"/>
+        </material>
+    </xacro:macro>
+    <xacro:macro name="material_red">
+        <material name="red">
+            <color rgba="1 0 0 0 1"/>
+        </material>
+    </xacro:macro>
+    <xacro:macro name="material_black">
+        <material name="black">
+            <color rgba="0.05 0.05 0.05 1"/>
+        </material>
+    </xacro:macro>
+    <xacro:macro name="material_silver">
+        <material name="silver">
+            <color rgba="0.5 0.5 0.5 1"/>
+        </material>
+    </xacro:macro>
 </robot>

File: obot_description/urdf/other_parts/drive_wheel_macro.xacro (robot description, xacro)
@@ -3,5 +3,5 @@
     <xacro:macro name="material_black">
         <material name="black">
-            <color rgba="0.1 0.1 0.1 1"/>
+            <color rgba="0.025 0.025 0.025 1"/>
         </material>
     </xacro:macro>
@@ -20,9 +20,4 @@
             <mu1>1.0</mu1>
             <mu2>1.0</mu2>
-            <!-- <kp>1000000</kp> -->
-            <!-- <kd>0.001</kd> -->
-            <!-- <minDepth>0.001</minDepth> -->
-            <!-- <fdir1>${fdir}</fdir1> -->
-            <material>Gazebo/FlatBlack</material>
         </gazebo>
     </xacro:macro>

File: obot_description/urdf/other_parts/drive_wheel_rim_macro.xacro (robot description, xacro)
@@ -51,10 +51,4 @@
             </visual>
         </link>
-        <!-- <gazebo reference="${base_name}">
-            <material>Gazebo/SkyBlue</material>
-        </gazebo> -->
-        <gazebo reference="${base_name}">
-            <material>Gazebo/Red</material>
-        </gazebo>
     </xacro:macro>
 </robot>

File: obot_description/urdf/robot_core.xacro (robot description, xacro)
@@ -1,5 +1,4 @@
 <?xml version="1.0"?>
 <robot xmlns:xacro="http://www.ros.org/wiki/xacro">
-    <xacro:include filename="other_parts/box_with_fillet_macro.xacro"/>
     <xacro:include filename="other_parts/drive_wheel_macro.xacro"/>
     <xacro:include filename="other_parts/drive_wheel_rim_macro.xacro"/>
@@ -11,5 +10,5 @@
     <xacro:property name="chassis_thickness" value="0.005"/>
     <xacro:property name="chassis_mass" value="2.0"/>
-    <xacro:property name="beam_height" value="0.05"/>
+    <xacro:property name="beam_height" value="0.06"/>
     <xacro:property name="beam_radius" value="0.005"/>
     <xacro:property name="chassis_color" value="orange"/>
@@ -37,5 +36,5 @@
             <cylinder radius="${chassis_radius}" length="${chassis_thickness}"/>
           </geometry>
-          <material name="${chassis_color}"/>
+          <xacro:material_orange/>
       </visual>
       <visual>
@@ -44,5 +43,5 @@
             <cylinder radius="${chassis_radius}" length="${chassis_thickness}"/>
           </geometry>
-          <material name="${chassis_color}"/>
+          <xacro:material_orange/>
       </visual>
       <visual>
@@ -51,5 +50,5 @@
             <cylinder radius="${chassis_radius}" length="${chassis_thickness}"/>
           </geometry>
-          <material name="${chassis_color}"/>
+          <xacro:material_orange/>
       </visual>
       <visual>
@@ -58,5 +57,5 @@
             <cylinder radius="${beam_radius}" length="${beam_height*2}"/>
           </geometry>
-          <material name="${chassis_color}"/>
+          <xacro:material_red/>
       </visual>
       <visual>
@@ -65,5 +64,5 @@
             <cylinder radius="${beam_radius}" length="${beam_height*2}"/>
           </geometry>
-          <material name="${chassis_color}"/>
+          <xacro:material_red/>
       </visual>
       <visual>
@@ -72,5 +71,5 @@
             <cylinder radius="${beam_radius}" length="${beam_height*2}"/>
           </geometry>
-          <material name="${chassis_color}"/>
+          <xacro:material_red/>
       </visual>
       <visual>
@@ -79,5 +78,5 @@
             <cylinder radius="${beam_radius}" length="${beam_height*2}"/>
           </geometry>
-          <material name="${chassis_color}"/>
+          <xacro:material_red/>
       </visual>
       <collision>
@@ -91,8 +90,4 @@
       </xacro:inertial_cylinder>
     </link>
-    <gazebo reference="chassis">
-        <!-- <material>Gazebo/DarkGrey</material> -->
-        <material>Gazebo/Orange</material>
-    </gazebo>
     <!--  ########################### -->
     <!-- LEFT DRIVE WHEEL -->
@@ -140,5 +135,5 @@
                 <sphere radius="${castor_wheel_radius}" />
             </geometry>
-            <material name="silver"/>
+            <xacro:material_silver/>
         </visual>
         <collision>
@@ -155,9 +150,4 @@
         <mu1>0.001</mu1>
         <mu2>0.001</mu2>
-        <!-- <kp>1000000.0</kp> -->
-        <!-- <kd>1.0</kd> -->
-        <!-- <fdir1>1 0 0</fdir1> -->
-        <!-- <minDepth>0.01</minDepth> -->
-        <material>Gazebo/Silver</material>
     </gazebo>
     <!--  ########################### -->

File: obot_description/urdf/robot_urdf.xacro (robot description, xacro)
@@ -4,4 +4,5 @@
     <xacro:include filename="inertia_macros.xacro" />
     <xacro:include filename="robot_core.xacro" />
-    <xacro:include filename="controllers/gazebo_control.xacro" />
+    <xacro:include filename="controllers/ign_gazebo_control.xacro" />
 </robot>
+<!-- xacro robot_urdf.xacro > _robot.urdf -->

File: obot_description/urdf/sensors/cam.xacro (robot description, xacro)
@@ -1,4 +1,9 @@
 <?xml version="1.0"?>
 <robot xmlns:xacro="http://www.ros.org/wiki/xacro" >
+    <xacro:macro name="material_black">
+        <material name="black">
+            <color rgba="0.025 0.025 0.025 1"/>
+        </material>
+    </xacro:macro>
     <xacro:macro name="insert_camera" params="base_name parent_name x y z mass width height min_range max_range tilt_angle visualize">
         <joint name="${base_name}_joint" type="fixed">
@@ -13,5 +18,5 @@
                     <cylinder radius="0.015" length="0.04"/>
                 </geometry>
-                <material name="grey"/>
+                <xacro:material_black/>
             </visual>
             <visual>
@@ -21,5 +26,5 @@
                     <box size="0.04 0.06 0.02"/>
                 </geometry>
-                <material name="grey"/>
+                <xacro:material_black/>
             </visual>
             <collision>
@@ -39,50 +44,7 @@
         </joint>
         <link name="${base_name}_optical_link"/>
-        <gazebo reference="${base_name}">
-          <material>Gazebo/DarkGrey</material>
-          <sensor name="${base_name}" type="camera">
-            <pose> 0 0 0 0 0 0 </pose>
-            <visualize>${visualize}</visualize>
-            <update_rate>20</update_rate>
-            <camera>
-                <!-- <horizontal_fov>1.089</horizontal_fov> -->
-                <horizontal_fov>1.46608</horizontal_fov>
-                <image>
-                    <format>R8G8B8</format>
-                    <width>${width}</width>
-                    <height>${height}</height>
-                </image>
-                <clip>
-                    <near>${min_range}</near>
-                    <far>${max_range}</far>
-                </clip>
-            </camera>
-            <plugin name="${base_name}_plugin" filename="libgazebo_ros_camera.so">
-                <frame_name>${base_name}_optical_link</frame_name>
-            </plugin>
-          </sensor>
-        </gazebo>
     </xacro:macro>
 </robot>
- <!-- <joint name="line_cam_joint" type="fixed">
-        <parent link="chassis"/>
-        <child link="line_cam"/>
-        <origin xyz="0.305 0 0.08" rpy="0 0 0"/>
-    </joint>
-    <link name="line_cam">
-        <visual>
-            <geometry>
-                <box size="0.010 0.03 0.03"/>
-            </geometry>
-            <material name="red"/>
-        </visual>
-    </link>
-    <joint name="line_cam_optical_joint" type="fixed">
-        <parent link="line_cam"/>
-        <child link="line_cam_link_optical"/>
-        <origin xyz="0 0 0" rpy="${-pi/2} 0 ${-pi/2}"/>
-    </joint>
-    <link name="line_cam_link_optical"></link>
-    <gazebo reference="line_cam">
+    <!-- <gazebo reference="line_cam">
         <material>Gazebo/Red</material>
         <sensor name="line_cam" type="camera">

File: obot_description/urdf/sensors/imu.xacro (robot description, xacro)
@@ -9,59 +9,10 @@
         <link name="${base_name}"/>
         <gazebo reference="${base_name}">
-            <sensor name="${base_name}" type="imu">
-                <always_on>true</always_on>
-                <update_rate>30</update_rate>
-                <visualize>true</visualize>
-                <imu>
-                    <angular_velocity>
-                        <x>
-                            <noise type="gaussian">
-                                <mean>0.0</mean>
-                                <stddev>2e-4</stddev>
-                            </noise>
-                        </x>
-                        <y>
-                            <noise type="gaussian">
-                                <mean>0.0</mean>
-                                <stddev>2e-4</stddev>
-                            </noise>
-                        </y>
-                        <z>
-                            <noise type="gaussian">
-                                <mean>0.0</mean>
-                                <stddev>2e-4</stddev>
-                            </noise>
-                        </z>
-                    </angular_velocity>
-                    <linear_acceleration>
-                        <x>
-                            <noise type="gaussian">
-                                <mean>0.0</mean>
-                                <stddev>1.7e-2</stddev>
-                            </noise>
-                        </x>
-                        <y>
-                            <noise type="gaussian">
-                                <mean>0.0</mean>
-                                <stddev>1.7e-2</stddev>
-                            </noise>
-                        </y>
-                        <z>
-                            <noise type="gaussian">
-                                <mean>0.0</mean>
-                                <stddev>1.7e-2</stddev>
-                            </noise>
-                        </z>
-                    </linear_acceleration>
-                </imu>
-                <plugin name="${base_name}_plugin" filename="libgazebo_ros_imu_sensor.so">
-                    <ros>
-                        <namespace>${base_name}</namespace>
-                        <remapping>~/out:=data</remapping>
-                    </ros>
-                    <initial_orientation_as_reference>false</initial_orientation_as_reference>
-                    <frame_name>${base_name}</frame_name>
-                </plugin>
-            </sensor>
+          <sensor name="${base_name}" type="imu">
+          <always_on>1</always_on>
+          <update_rate>1</update_rate>
+          <visualize>true</visualize>
+          <topic>${base_name}</topic>
+          </sensor>
         </gazebo>
     </xacro:macro>

File: obot_description/urdf/sensors/lidar.xacro (robot description, xacro)
@@ -1,4 +1,9 @@
 <?xml version="1.0"?>
 <robot xmlns:xacro="http://www.ros.org/wiki/xacro" >
+    <xacro:macro name="material_black">
+        <material name="black">
+            <color rgba="0.025 0.025 0.025 1"/>
+        </material>
+    </xacro:macro>
     <xacro:macro name="insert_lidar" params="base_name parent_name x y z mass samples min_angle max_angle min_range max_range visualize">
         <joint name="${base_name}_joint" type="fixed">
@@ -13,5 +18,5 @@
                     <cylinder radius="0.03" length="0.04"/>
                 </geometry>
-                <material name="grey"/>
+                <xacro:material_black/>
             </visual>
             <collision>
@@ -26,32 +31,32 @@
         </link>
         <gazebo reference="${base_name}">
-            <material>Gazebo/DarkGrey</material>
-            <sensor name="${base_name}" type="ray">
-                <pose> 0 0 0 0 0 0 </pose>
-                <visualize>${visualize}</visualize>
-                <update_rate>10</update_rate>
-                <ray>
-                    <scan>
-                        <horizontal>
-                            <samples>${samples}</samples>
-                            <min_angle>${min_angle}</min_angle>
-                            <max_angle>${max_angle}</max_angle>
-                        </horizontal>
-                    </scan>
-                    <range>
-                        <min>${min_range}</min>
-                        <max>${max_range}</max>
-                    </range>
-                </ray>
-                <plugin name="${base_name}_plugin" filename="libgazebo_ros_ray_sensor.so">
-                    <ros>
-                        <namespace>${base_name}</namespace>
-                        <remapping>~/out:=scan</remapping>
-                        <!-- <argument>~/out:=scan</argument> -->
-                    </ros>
-                    <output_type>sensor_msgs/LaserScan</output_type>
-                    <frame_name>${base_name}</frame_name>
-                </plugin>
-            </sensor>
+          <sensor name='${base_name}' type='gpu_lidar'>
+            <pose>0 0 0 0 0 0</pose>
+            <topic>${base_name}</topic>
+            <update_rate>10</update_rate>
+            <ray>
+              <scan>
+                <horizontal>
+                  <samples>${samples}</samples>
+                  <min_angle>${min_angle}</min_angle>
+                  <max_angle>${max_angle}</max_angle>
+                  <resolution>0.5</resolution>
+                </horizontal>
+                <vertical>
+                  <samples>1</samples>
+                  <resolution>0.01</resolution>
+                  <min_angle>0</min_angle>
+                  <max_angle>0</max_angle>
+                </vertical>
+              </scan>
+              <range>
+                <min>${min_range}</min>
+                <max>${max_range}</max>
+                <resolution>0.01</resolution>
+              </range>
+            </ray>
+            <always_on>1</always_on>
+            <visualize>${visualize}</visualize>
+          </sensor>
         </gazebo>
     </xacro:macro>

File: obot_description/urdf/sensors/sonar.xacro (robot description, xacro)
@@ -1,7 +1,9 @@
 <?xml version="1.0"?>
 <robot xmlns:xacro="http://www.ros.org/wiki/xacro">
-    <!-- <xacro:arg name="sonar_visual"   default="false"/> -->
-    <!-- <xacro:property name="deg2rad" value="0.017460317"/>
-    <xacro:property name="scan_angle" value="1"/> -->
+    <xacro:macro name="material_blue">
+        <material name="blue">
+            <color rgba="0.2 0.2 1 1"/>
+        </material>
+    </xacro:macro>
     <xacro:macro name="insert_sonar" params="base_name parent_name x y z rx ry rz mass min_range max_range resolution visualize">
         <joint name="${base_name}_joint" type="fixed">
@@ -16,5 +18,5 @@
                     <cylinder radius="0.006" length="0.006"/>
                 </geometry>
-                <material name="blue"/>
+                <xacro:material_blue/>
             </visual>
             <collision>
@@ -29,5 +31,5 @@
                     <cylinder radius="0.006" length="0.006"/>
                 </geometry>
-                <material name="blue"/>
+                <xacro:material_blue/>
             </visual>
             <collision>
@@ -41,43 +43,4 @@
             </xacro:inertial_cylinder>
         </link>
-        <gazebo reference="${base_name}">
-            <material>Gazebo/Blue</material>
-            <sensor name="${base_name}" type="ray">
-                <always_on>true</always_on>
-                <visualize>${visualize}</visualize>
-                <pose>0.0 0 0.0 0 0 0</pose>
-                <update_rate>5</update_rate>
-                <ray>
-                    <scan>
-                        <horizontal>
-                            <samples>20</samples>
-                            <resolution>1</resolution>
-                            <min_angle>${-pi/90}</min_angle>
-                            <max_angle>${pi/90}</max_angle>
-                        </horizontal>
-                        <vertical>
-                            <samples>20</samples>
-                            <resolution>1</resolution>
-                            <min_angle>${-pi/150}</min_angle>
-                            <max_angle>${pi/150}</max_angle>
-                        </vertical>
-                    </scan>
-                    <range>
-                        <min>${min_range}</min>
-                        <max>${max_range}</max>
-                        <resolution>${resolution}</resolution>
-                    </range>
-                </ray>
-                <plugin name="${base_name}_plugin" filename="libgazebo_ros_ray_sensor.so">
-                    <ros>
-                        <namespace>${base_name}</namespace>
-                        <remapping>~/out:=range</remapping>
-                    </ros>
-                    <output_type>sensor_msgs/Range</output_type>
-                    <radiation_type>ultrasound</radiation_type>
-                    <frame_name>${base_name}</frame_name>
-                </plugin>
-            </sensor>
-        </gazebo>
     </xacro:macro>
 </robot>
